File: Eagle/Jerry_microMouse.sch (EAGLE design)
At the start: 61 parts, among them IC1 DSPIC33FJ64MC804-PT, IC2 L293D, IC3 LM340MP-5.0, IC4 LM3940IMP-3.3

Commit message: update PCB, manually routing
Parts:
- removed FREE_PINS: (no value), con-lstb:MA03-1
- added C13, C9: 100nF, rcl:C-EUC0805
- added FREE_PINS1: (no value), con-lstb:MA03-1
- added FREE_PINS2: (no value), con-lstb:MA04-1
Connections:
- net N$2 renamed RM_M+
- net N$4 renamed LM_M+
- net N$6 renamed RM_M-
- net N$7 renamed LM_M-
- new net BUZZER: BUZZER.2, IC1.PWM1H2/DAC1RP/RP12/CN14/PMD0/RB12
- new net N$26: FREE_PINS2.4, IC1.RP20/CN25/PMA4/RC4
- new net N$27: FREE_PINS1.2, IC1.TMS/PMA10/RA10
- new net N$28: FREE_PINS1.1, IC1.TCK/PMA7/RA7
- net +5V: now also C12.2, IC4.IN
- net +9V: no longer C12.2, IC4.IN
- net GND: now also C13.2, C9.2
- net LM_H_BRDG_DIR_1: now also IC1.RP24/CN20/PMA5/RC8; no longer IC1.PWM1H2/DAC1RP/RP12/CN14/PMD0/RB12
- net LM_H_BRDG_DIR_2: now also IC1.RP25/CN19/PMA6/RC9; no longer IC1.PWM1L2/DAC1RN/RP13/CN13/PMRD/RB13
- net N$1: now also IC1.PWM2L1/RP23/CN17/PMA0/RC7; no longer IC1.RP24/CN20/PMA5/RC8
- net N$21: now also FREE_PINS1.3, IC1.PWM1L2/DAC1RN/RP13/CN13/PMRD/RB13; no longer BUZZER.2, IC1.RP20/CN25/PMA4/RC4
- net N$22: now also FREE_PINS2.1; no longer FREE_PINS.1
- net N$23: now also FREE_PINS2.2; no longer FREE_PINS.2
- net N$24: now also FREE_PINS2.3; no longer FREE_PINS.3
- net RM_ENC_CH_A: now also IC1.AN4/C1IN-/RP2/CN6/RB2; no longer IC1.AN7/RP17/CN9/RC1
- net RM_ENC_CH_B: now also IC1.AN5/C1IN+/RP3/CN7/RB3; no longer IC1.AN6/RP16/CN8/RC0
- net RM_H_BRDG_DIR_1: now also IC1.AN7/RP17/CN9/RC1; no longer IC1.AN5/C1IN+/RP3/CN7/RB3
- net RM_H_BRDG_DIR_2: now also IC1.AN6/RP16/CN8/RC0; no longer IC1.AN4/C1IN-/RP2/CN6/RB2
- net UART2_RX: now also IC1.SCL1/RP8/CN22/PMD4/RB8; no longer IC1.INT0/RP7/CN23/PMD5/RB7
- net UART2_TX: now also IC1.INT0/RP7/CN23/PMD5/RB7; no longer IC1.SCL1/RP8/CN22/PMD4/RB8
- net VDD: now also C13.1, C9.1
Other:
- moved on the sheet: 9V-INPUT-1, 9V-INPUT-2, C3, D3, D4, LED1, LED2, R1, R2
